File: rx5808_4button.sch (KiCad schematic (older format))
At the start: 61 parts, among them IC1 ATMEGA328-A, P1 CONN_01X02, P10 CONN_01X01, P11 CONN_01X01, P2 CONN_01X05, P3 CONN_02X03, P4 CONN_01X02, P5 BNC, P6 BNC, P7 CONN_01X02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

Commit message: das neue Immersion RC RaceBand kommt zum Empfänger dazu!
Parts:
- C1, C10, C11, C12, C13, C2, C3, C4, C5, C6, C7, C8, C9: symbol C -> C-RESCUE-rx5808_4button
- D1: value SB130 -> B 140 F
- D2: value TVS 18V -> P6SMB 18A SMD
- R1, R10, R11, R12, R13, R14, R15, R16, R17, R18, R19, R2, R20, R21, R22, R3, R4, R5, R6, R7, R8, R9: symbol R -> R-RESCUE-rx5808_4button
Changed lines of the file:
@@
 EESchema Schematic File Version 2
+LIBS:rx5808_4button-rescue
 LIBS:SMA_EDGE
 LIBS:power
@@
 $EndComp
 $Comp
-L C C2
+L C-RESCUE-rx5808_4button C2
 U 1 1 54EE2194
 P 2450 3700
@@
 $EndComp
 $Comp
-L C C4
+L C-RESCUE-rx5808_4button C4
 U 1 1 54EE231F
 P 2850 3700
@@
 $EndComp
 $Comp
-L C C6
+L C-RESCUE-rx5808_4button C6
 U 1 1 54EE23A2
 P 3250 3700
@@
 $EndComp
 $Comp
-L C C7
+L C-RESCUE-rx5808_4button C7
 U 1 1 54EE23B4
 P 3650 3700
@@
 buzzer
 $Comp
-L R R6
+L R-RESCUE-rx5808_4button R6
 U 1 1 54EE241A
 P 4750 4800
@@
 $EndComp
 $Comp
-L R R4
+L R-RESCUE-rx5808_4button R4
 U 1 1 54EE248C
 P 4750 4600
@@
 $EndComp
 $Comp
-L R R5
+L R-RESCUE-rx5808_4button R5
 U 1 1 54EE24A3
 P 4750 4700
@@
 NoConn ~ 2050 5850
 $Comp
-L C C1
+L C-RESCUE-rx5808_4button C1
 U 1 1 54EE2578
 P 1550 5000
@@
 Gayduino\nProgrammierstecker
 $Comp
-L R R3
+L R-RESCUE-rx5808_4button R3
 U 1 1 54EE2F7B
 P 4750 4500
@@
 	4500 4500 3950 4500
 $Comp
-L R R9
+L R-RESCUE-rx5808_4button R9
 U 1 1 54EE3190
 P 4750 6700
@@
 	5950 4850 5950 5100
 $Comp
-L C C8
+L C-RESCUE-rx5808_4button C8
 U 1 1 54EE3CF9
 P 4500 5850
@@
 	800  6150 800  5850
 $Comp
-L R R7
+L R-RESCUE-rx5808_4button R7
 U 1 1 54EE5131
 P 4750 6000
@@
 $EndComp
 $Comp
-L R R8
+L R-RESCUE-rx5808_4button R8
 U 1 1 54EE52EF
 P 4750 6100
@@
 5,8GHz Antenne
 $Comp
-L C C11
+L C-RESCUE-rx5808_4button C11
 U 1 1 54EE66EB
 P 5900 3400
@@
 $EndComp
 $Comp
-L C C12
+L C-RESCUE-rx5808_4button C12
 U 1 1 54EE66FD
 P 6300 3400
@@
 $EndComp
 $Comp
-L R R1
+L R-RESCUE-rx5808_4button R1
 U 1 1 54EE6E06
 P 4150 3650
@@
 P 1400 1100
 F 0 "D1" H 1400 1200 50  0000 C CNN
-F 1 "SB130" H 1400 1000 50  0000 C CNN
+F 1 "B 140 F" H 1400 1000 50  0000 C CNN
 F 2 "Diodes_SMD:Diode-SMA_Standard" H 1400 1100 60  0001 C CNN
 F 3 "" H 1400 1100 60  0000 C CNN
@@
 	4500 1100 6400 1100
 $Comp
-L R R2
+L R-RESCUE-rx5808_4button R2
 U 1 1 54EE86C7
 P 4250 1400
@@
 Connection ~ 4600 1200
 $Comp
-L R R10
+L R-RESCUE-rx5808_4button R10
 U 1 1 54EE87EC
 P 4800 1350
@@
 $EndComp
 $Comp
-L R R11
+L R-RESCUE-rx5808_4button R11
 U 1 1 54EE881D
 P 4800 1850
@@
 Connection ~ 4600 1100
 $Comp
-L C C9
+L C-RESCUE-rx5808_4button C9
 U 1 1 54EE89CE
 P 5200 1300
@@
 $EndComp
 $Comp
-L C C10
+L C-RESCUE-rx5808_4button C10
 U 1 1 54EE8A62
 P 6400 1300
@@
 $EndComp
 $Comp
-L C C3
+L C-RESCUE-rx5808_4button C3
 U 1 1 54EE948B
 P 2600 2300
@@
 $EndComp
 $Comp
-L C C5
+L C-RESCUE-rx5808_4button C5
 U 1 1 54EE9497
 P 3000 2300
@@
 P 1600 1450
 F 0 "D2" H 1600 1550 50  0000 C CNN
-F 1 "TVS 18V" H 1600 1350 50  0000 C CNN
+F 1 "P6SMB 18A SMD" H 1600 1350 50  0000 C CNN
 F 2 "Diodes_SMD:Diode-SMB_Standard" H 1600 1450 60  0001 C CNN
 F 3 "" H 1600 1450 60  0000 C CNN
@@
 $EndComp
 $Comp
-L R R12
+L R-RESCUE-rx5808_4button R12
 U 1 1 54EEC7A1
 P 9050 1400
@@
 $EndComp
 $Comp
-L R R13
+L R-RESCUE-rx5808_4button R13
 U 1 1 54F075A5
 P 7250 5050
@@
 $EndComp
 $Comp
-L R R14
+L R-RESCUE-rx5808_4button R14
 U 1 1 54F07909
 P 7400 5050
@@
 $EndComp
 $Comp
-L R R15
+L R-RESCUE-rx5808_4button R15
 U 1 1 54F079CF
 P 8250 5050
@@
 $EndComp
 $Comp
-L R R16
+L R-RESCUE-rx5808_4button R16
 U 1 1 54F079DB
 P 8400 5050
@@
 $EndComp
 $Comp
-L R R17
+L R-RESCUE-rx5808_4button R17
 U 1 1 54F07BA1
 P 9250 5050
@@
 $EndComp
 $Comp
-L R R18
+L R-RESCUE-rx5808_4button R18
 U 1 1 54F07BAD
 P 9400 5050
@@
 $EndComp
 $Comp
-L R R19
+L R-RESCUE-rx5808_4button R19
 U 1 1 54F07BB9
 P 10250 5050
@@
 $EndComp
 $Comp
-L R R20
+L R-RESCUE-rx5808_4button R20
 U 1 1 54F07BC5
 P 10400 5050
@@
 $EndComp
 $Comp
-L C C13
+L C-RESCUE-rx5808_4button C13
 U 1 1 54F19297
 P 5800 1300
@@
 $EndComp
 $Comp
-L R R21
+L R-RESCUE-rx5808_4button R21
 U 1 1 54F19CCA
 P 1500 2450
@@
 extra RSSI Ausgang\nfür Toni
 $Comp
-L R R22
+L R-RESCUE-rx5808_4button R22
 U 1 1 551FF942
 P 4950 1850
