File: DiversityModule/diversityModule.kicad_pcb (KiCad board)
At the start: 2 copper layers, 56.5 x 25 mm, 44 parts, among them IC1 LP38798, IC2 TDA1308A, P1 CONN_02X05, P2 CONN_01X03, Q1 BFP840, U1 sn74lvc1g3157, U2 RX5808

Commit message: BOM hinzugefügt
Changed lines of the file:
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@@
-(kicad_pcb (version 4) (host pcbnew "(2016-06-07 BZR 6887)-product")
+(kicad_pcb (version 4) (host pcbnew "(2016-07-18 BZR 6982)-product")
   (general
     (links 106)
@@
   )
   (setup
-    (last_trace_width 0.3)
+    (last_trace_width 0.786937)
     (user_trace_width 0.15)
     (user_trace_width 0.2)
@@
     (user_trace_width 0.786937)
     (trace_clearance 0.2)
-    (zone_clearance 0.2)
+    (zone_clearance 0.23)
     (zone_45_only no)
     (trace_min 0.15)
@@
   (segment (start 101.5 90.05) (end 101.5 91) (width 0.15) (layer F.Cu) (net 16))
   (segment (start 105.9 90.55) (end 105.9 90.6) (width 0.15) (layer F.Cu) (net 16))
-  (segment (start 98.25 87.2) (end 98.25 85.65) (width 0.5) (layer F.Cu) (net 17))
+  (segment (start 98.25 87.2) (end 98.25 85.65) (width 0.786937) (layer F.Cu) (net 17))
   (segment (start 95.044 86.67) (end 96.57 86.67) (width 0.25) (layer F.Cu) (net 17))
   (segment (start 96.57 86.67) (end 97.1 87.2) (width 0.25) (layer F.Cu) (net 17))
@@
   (segment (start 138.06 97.78) (end 136.01 97.78) (width 0.3) (layer B.Cu) (net 33))
   (segment (start 136.01 97.78) (end 135.1 98.69) (width 0.3) (layer B.Cu) (net 33))
-  (segment (start 98.25 84.55) (end 98.25 83.1) (width 0.5) (layer F.Cu) (net 34))
+  (segment (start 98.25 84.55) (end 98.25 83.1) (width 0.786937) (layer F.Cu) (net 34))
   (zone (net 5) (net_name /+3,0V) (layer F.Cu) (hatch edge 0.508)
     (priority 3)
@@
   (zone (net 2) (net_name GNDA) (layer B.Cu) (hatch edge 0.508)
     (priority 2)
-    (connect_pads (clearance 0.15))
+    (connect_pads (clearance 0.23))
     (min_thickness 0.2)
     (fill yes (arc_segments 32) (thermal_gap 0.508) (thermal_bridge_width 1.016))
@@
         (xy 116 94.5) (xy 116 96) (xy 117.5 96) (xy 117.5 100.5) (xy 115.5 102)
         (xy 111.5 102) (xy 111 101.5) (xy 111 98.5) (xy 105 92.5) (xy 91 92.5)
-        (xy 91 79.5) (xy 111.5 79.5) (xy 111.5 84)
+        (xy 91 79.5) (xy 111.5 79.5)
       )
     )
@@
         (xy 116 94.5) (xy 116 96) (xy 117.5 96) (xy 117.5 100.5) (xy 115.5 102)
         (xy 111.5 102) (xy 111 101.5) (xy 111 98.5) (xy 105 92.5) (xy 91 92.5)
-        (xy 91 79.5) (xy 111.5 79.5) (xy 111.5 84)
+        (xy 91 79.5) (xy 111.5 79.5)
       )
     )
@@
         (xy 110.5 101.5) (xy 111.5 102.5) (xy 116 102.5) (xy 118 101) (xy 118 86.5)
         (xy 116 86.5) (xy 116 83.5) (xy 112 83.5) (xy 112 79.5) (xy 149 79.5)
-        (xy 149 105.5)
       )
     )
@@
         (xy 110.5 101.5) (xy 111.5 102.5) (xy 116 102.5) (xy 118 101) (xy 118 86.5)
         (xy 116 86.5) (xy 116 83.5) (xy 112 83.5) (xy 112 79.5) (xy 149 79.5)
-        (xy 149 105.5)
       )
     )
