File: Platine/rx5808_4button.kicad_pcb (KiCad board)
At the start: 2 copper layers, 50 x 29.5 mm, 54 parts, among them IC1 ATMEGA328-A, P1 CONN_01X04, P2 CONN_01X05, P6 CONN_01X04, P7 CONN_02X05, U1 TPS62160, U2 RX5808, U3 sn74lvc1g3157, U4 MCPL3-BC-V, Y1 16 MHz

Commit message: BOM fertiggestellt und alten Code gelöscht
Changed lines of the file:
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@@
   )
   (layers
-    (0 F.Cu signal)
-    (31 B.Cu signal)
-    (34 B.Paste user)
+    (0 F.Cu signal hide)
+    (31 B.Cu signal hide)
+    (34 B.Paste user hide)
     (35 F.Paste user)
-    (36 B.SilkS user)
+    (36 B.SilkS user hide)
     (37 F.SilkS user)
-    (38 B.Mask user)
+    (38 B.Mask user hide)
     (39 F.Mask user)
-    (40 Dwgs.User user)
-    (42 Eco1.User user)
-    (44 Edge.Cuts user)
+    (40 Dwgs.User user hide)
+    (42 Eco1.User user hide)
+    (44 Edge.Cuts user hide)
   )
   (setup
@@
     (mod_text_size 1 1)
     (mod_text_width 0.15)
-    (pad_size 1.6 3.4)
+    (pad_size 1.59766 1.80086)
     (pad_drill 0)
     (pad_to_mask_clearance 0.1)
     (aux_axis_origin 0 0)
-    (visible_elements FFFEEF39)
+    (visible_elements FFFEEB39)
     (pcbplotparams
-      (layerselection 0x00080_7ffffffe)
+      (layerselection 0x00008_7ffffffe)
       (usegerberextensions false)
       (excludeedgelayer false)
@@
     (fp_line (start -2.5 1.25) (end 2.5 1.25) (layer F.CrtYd) (width 0.05))
     (fp_line (start 2.5 1.25) (end 2.5 -1.25) (layer F.CrtYd) (width 0.05))
-    (pad 2 smd rect (at 1.41986 0 180) (size 1.59766 1.80086) (layers F.Cu F.Mask)
+    (pad 2 smd rect (at 1.41986 0 180) (size 1.59766 1.80086) (layers F.Cu F.Paste F.Mask)
       (net 52 "Net-(D5-Pad2)"))
     (pad 1 smd rect (at -1.41986 0 180) (size 1.59766 1.80086) (layers F.Cu F.Mask)
@@
     (descr " NR3015")
     (tags " NR3015T2R2M")
-    (fp_text reference L1 (at -3.25 7.25 90) (layer F.SilkS)
-      (effects (font (size 1 1) (thickness 0.15)))
-    )
+    (fp_text reference L1 (at 0 2.25 90) (layer F.SilkS)
+      (effects (font (size 1 1) (thickness 0.15)))
+    )
